Commit message: Tow model comparaison

File: install/vis_nav/share/vis_nav/description/urdf/scout_robot.urdf (robot description, URDF)
Before this commit: robot scout, 10 links, 9 joints
Links:
- added link cameraFishEye, mass 1e-5; collision cylinder length=0.03 radius=0.03; visual cylinder length=0.03 radius=0.03
- added link fisheye_frame
Joints:
- added joint base_link_cameraFishEye_joint: type fixed, parent base_link, child cameraFishEye, origin xyz=0.21 0 0.5 rpy=0 0 0, axis 0.19 0 0.5
- added joint fisheye_joint: type fixed, parent cameraFishEye, child fisheye_frame, origin xyz=0 0 0 rpy=-1.57 0 -1.57
