Commit message: Final changes

File: src/vis_nav/description/urdf/robot_w.urdf (robot description, URDF)
Before this commit: robot robot, 33 links, 32 joints
Links:
- removed link caster_wheel1
- removed link caster_wheel2
- added link front_laser, mass 1e-5; collision box size=0.1 0.1 0.1; visual cylinder length=0.02 radius=0.025
- added link front_left, mass 0.1; collision cylinder length=0.025 radius=0.0335; visual cylinder length=0.025 radius=0.0335
- added link front_right, mass 0.1; collision cylinder length=0.025 radius=0.0335; visual cylinder length=0.025 radius=0.0335
- link batterie: mass 0.1546875 -> 0.5
- link rear_left: mass 0.044070654 -> 0.1
- link rear_right: mass 0.044070654 -> 0.1
Joints:
- removed joint caster_wheel1_joint
- removed joint caster_wheel2_joint
- added joint base_link_front_laser_joint: type fixed, parent base_link, child front_laser, origin xyz=0.25 0 0.13 rpy=0 0 0, axis 0 0 1
- added joint front_left_wheel_joint: type continuous, parent base_link, child front_left, origin xyz=0.1775 0.0625 0.0335 rpy=-1.5707963267948966 0 0, axis 0 0 1
- added joint front_right_wheel_joint: type continuous, parent base_link, child front_right, origin xyz=0.1775 -0.0625 0.0335 rpy=1.5707963267948966 0 0, axis 0 0 -1
- joint rear_left_wheel_joint: origin xyz=0.0 0.065 -0.02 rpy=-1.5707963267948966 0 0 -> xyz=0.0825 0.0625 0.0335 rpy=-1.5707963267948966 0 0; parent chassis2 -> base_link
- joint rear_right_wheel_joint: origin xyz=0.0 -0.065 -0.02 rpy=1.5707963267948966 0 0 -> xyz=0.0825 -0.0625 0.0335 rpy=1.5707963267948966 0 0; parent chassis2 -> base_link
